File: 00-produccion-pcbs/1-versiones-profes/grupo-02/g-02-sec-02-rev-a/g-02-sec-02-rev-a.kicad_pcb (KiCad board)
At the start: 2 copper layers, 100 x 100 mm, 68 parts, among them J10 AudioJack2_SwitchT, J11 AudioJack2_SwitchT, J12 AudioJack2_SwitchT, J13 AudioJack2_SwitchT, J14 AudioJack2_SwitchT, J2 Barrel_Jack_Switch, J4 Barrel_Jack_Switch, J6 AudioJack2_SwitchT, J7 AudioJack2_SwitchT, J8 AudioJack2_SwitchT, J9 AudioJack2_SwitchT, Q1 BC548, Q10 PN2222A, Q3 PN2222A, Q4 PN2222A, Q5 PN2222A, Q6 PN2222A, Q7 PN2222A, Q8 PN2222A, Q9 PN2222A, SW4 SW_SPDT, U2 4015, U4 L7805

Commit message: corregido 02-02
Other:
- board text added: "g-02-sec-02-rev-a"
Changed lines of the file:
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@@
 		(layer "Edge.Cuts")
+	)
+	(gr_text "g-02-sec-02-rev-a"
+		(at 119.359068 57.176757 0)
+		(layer "F.SilkS")
+		(effects
+			(font
+				(size 1.5 1.5)
+				(thickness 0.3)
+				(bold yes)
+			)
+			(justify left bottom)
+		)
 	)
 	(segment
