File: 00-produccion-pcbs/1-versiones-profes/grupo-04/g-04-osc-01-rev-a/g-04-osc-01-rev-a.kicad_pcb (KiCad board)
At the start: 2 copper layers, 100 x 80 mm, 35 parts, among them J1 Barrel_Jack_Switch, J3 Barrel_Jack_Switch, J4 AudioJack2_SwitchT, J5 Conn_01x03_Pin, SW3 SW_SPDT, U1 40106, U2 L7805, U3 LM324

Commit message: uploaded g-04-01
Parts:
- added R8: 1K, Resistor_THT:R_Axial_DIN0207_L6.3mm_D2.5mm_P10.16mm_Horizontal, F.Cu at (206.9, 101.5)
Connections:
- J4 pad 1: unconnected-(J4-Pad1) -> GND
- J4 pad 3: unconnected-(J4-Pad3) -> OUTPUT
- U3 pad 1: OUTPUT -> Net-(U3A--)
- U3 pad 2: OUTPUT -> Net-(U3A--)
Routing:
- net Net-(D1-A): track 66.7 -> 32.3 mm, vias 0 -> 1
- net Net-(U3A--): track 0.00 -> 26.8 mm
- net GND: track 0.00 -> 11.9 mm, vias 0 -> 2
- net +12V: track 100.1 -> 90.1 mm, vias 0 -> 3
- net +5V: track 131.9 -> 122.8 mm, vias 0 -> 1
- net OUTPUT: track 0.00 -> 7.67 mm
- net unconnected-(RV2-Pad3): vias 1 -> 0
Other:
- board text added: "g-04-osc-01-rev-a"
