File: 00-produccion-pcbs/1-versiones-profes/grupo-04/g-04-osc-01-rev-a/g-04-osc-01-rev-a.kicad_sch (KiCad schematic)
At the start: 42 parts, among them J1 Barrel_Jack_Switch, J3 Barrel_Jack_Switch, J4 AudioJack2_SwitchT, J5 Conn_01x03_Pin, SW3 SW_SPDT, U1 40106, U2 L7805, U3 LM324, U4 LM386

Commit message: uploaded g-04-01
Parts:
- removed C5, C7, C8: 10u, symbol Device:C_Polarized
- removed C6: 100n, symbol Device:C
- removed LS1: Speaker, symbol Device:Speaker
- removed RV6: 100K, symbol Device:R_Potentiometer
- removed U4: LM386, symbol Amplifier_Audio:LM386
- added R8: 1K, Resistor_THT:R_Axial_DIN0207_L6.3mm_D2.5mm_P10.16mm_Horizontal, symbol Device:R
Connections:
- net GND: now also J4.1
- net OUTPUT: now also J4.3, R8.1; no longer U3.1, U3.2 (-)
- new net: R8.2, U3.1, U3.2 (-)
- no-connect marks 12 -> 8
Other:
- note removed: "cambiar numero de pines a este orden (reemplazar T/TN/S)"
- moved on the sheet: J4
